File: PCB/esc.kicad_sch (KiCad schematic)
At the start: 31 parts, among them J1 Conn_01x04_Pin, J2 Conn_01x01, J3 Conn_01x01, J4 Conn_01x01, J5 Conn_01x01, J6 Conn_01x01, SW1 SW_SPST, U1 STM32C031K6T6, U2 TLV76133DCY, U3 LMV324A, U4 INA180A3

Commit message: Swapped opamp
Desgin now specifies an opamp with rail-to-rail input.
Parts:
- removed U3: LMV324A, Package_SO:TSSOP-14_4.4x5mm_P0.65mm, symbol Amplifier_Operational:LMV324
- added U3: TLV9064, Package_SO:TSSOP-14_4.4x5mm_P0.65mm, symbol Amplifier_Operational:TLV9064
Connections:
- net +3V3: now also U3.4 (V+)
- net GND: now also U3.11 (V-)
- net i_sense: now also U3.3 (+)
- net i_sense_buf: now also U3.1
- net v_a: now also U3.12 (+)
- net v_a_buf: now also U3.13 (-), U3.14
- net v_b: now also U3.10 (+)
- net v_b_buf: now also U3.8, U3.9 (-)
- net v_c: now also U3.5 (+)
- net v_c_buf: now also U3.6 (-), U3.7
- net at R2.1, R3.1: now also U3.2 (-)
